File: hardware/jnode/jnode_v32.brd (EAGLE design)
At the start: 55.8 x 18 mm, 63 parts, among them IC1 JENNIC_JN5139, IC2 ATMEGA32U4-AUQFN44, IC3 LTC3553, IC4 LSM303DLM, IC5 L3G4200D, IC6 MPL115A, SW1 SONDER_H_VIBRATIONSSCHALTER, T1 DMP2104LP-7, X1 USB-MICROB

Commit message: cc3000 wifi board for jnode
Parts:
- removed C13: 10µF, sparkfun:0603-CAP
- removed C15: 4.7µF, sparkfun:0402-CAP
- removed C16: 0.22µF, sparkfun:0402-CAP
- removed IC4: LSM303DLM, jnode:LGA28
- removed IC5: L3G4200D, sparkfun:LGA16-4X4
- removed R1: 10k, sparkfun:0402-RES
- added U$2: LSM9D, jnode:LGA4X4
- added U1: SHT21, zittel:DFN300X300X110-7N
- C11: value 10nF -> 0.22µF
- C2: value 0.1µF -> 100nF
- C3: value 470nF -> 4.7µF
- IC1: value JENNIC_JN5139 -> (none)
- MICRO_SD1: value SENSOR_BOARD_MOLEX_47309-2651'NEW' -> (none)
- R13: device sparkfun:0805 -> sparkfun:0402-RES
- X1: value USB-MICROB -> USBMICROB-XT; device sparkfun:USB-MICROB -> sparkfun:USB-MICROB-XT
- moved U$9 10.2 mm to (16.7, 10.2), turned to 270 degrees
- moved C8 9.36 mm to (22.8, 4.15)
- moved C9 8.56 mm to (22.8, 5.65)
- moved C11 2.87 mm to (26.3, 9.65), turned to 90 degrees
- moved U$1 2.54 mm to (48.3, 12.7)
- moved C3 2.44 mm to (25.2, 11.8), turned to 0 degrees
- moved C2 2.26 mm to (19.5, 4.20)
- moved R16 0.35 mm to (21.9, 1.80)
- moved C5 0.30 mm to (22.4, 14.4)
- moved BTN_PWR 0.22 mm to (55.5, 11.6)
- moved JP1 0.10 mm to (29.3, 2.50)
- turned C6 to 270 degrees
Connections:
- removed net N$25: C15.2, IC4.15
- removed net N$26: C11.2, C3.1, IC5.14
- removed net N$27: C3.2, R1.1
- removed net SHWO: IC2.13, JP1.2
- new net ATMEGARESET: IC1.11, IC2.13, JP1.2
- new net BLE_RES: IC2.25
- new net N$7: C11.2, U$2.P$8
- net 3G_INT2: now also U$2.P$13; no longer IC5.6
- net GND: now also C2.1, C3.2, C8.2, C9.1, U$2.P$22, U$2.P$23, U$2.P$5, U$2.P$6, U1.2; no longer C11.1, C13.1, C15.1, C2.2, C8.1, C9.2, IC4.1, IC4.17, IC4.2, IC4.28, IC4.3, IC4.4, IC5.10, IC5.11, IC5.12, IC5.13, IC5.4, IC5.8, IC5.9, R1.2
- net N$2: now also C3.1, U$2.P$7; no longer C16.1, IC4.16
- net N$8: now also C11.1, U$2.P$9; no longer C16.2, IC4.12
- net SCLK: now also U$2.P$21, U1.6; no longer IC4.20, IC4.24, IC5.2
- net SDAT: now also U$2.P$24, U1.1; no longer IC4.19, IC4.25, IC5.3
- net SSEL: now also IC1.12; no longer IC1.10
- net VCC: now also C2.2, U1.5
- net VSENS: now also C8.1, C9.2, U$2.P$10, U$2.P$15, U$2.P$16, U$2.P$17, U$2.P$18, U$2.P$19, U$2.P$20; no longer C13.2, C2.1, C8.2, C9.1, IC4.22, IC4.23, IC4.6, IC4.7, IC5.1, IC5.15, IC5.16, IC5.5
Routing:
- net GND: track 15.4 -> 39.9 mm, vias 43 -> 53
- net VCC: track 105.0 -> 114.6 mm
- net MISO: track 32.6 -> 23.5 mm, vias 4 -> 3
- net ATMEGARESET: track 0.00 -> 8.01 mm
- net SHWO: track 5.48 -> 0.00 mm
- net SDAT: track 50.6 -> 45.2 mm
- net N$9: track 26.9 -> 22.3 mm
- net VSENS: track 60.2 -> 56.0 mm, vias 6 -> 2
- net N$2: track 5.80 -> 1.89 mm
- net PBSTAT: track 58.8 -> 54.9 mm
- net VOUT: track 33.7 -> 37.1 mm
- net N$26: track 3.00 -> 0.00 mm
- net SSEL: track 38.7 -> 36.2 mm
- net N$25: track 1.97 -> 0.00 mm
- net SCLK: track 51.3 -> 49.8 mm
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- removed copper zone on layer 16, net VSENS
Other:
- board text added: "BTN_PWR"
- board text added: "IC2"
- board text added: "IC3"
- board text added: "L1"
- board text added: "LED1"
- board text added: "LED2"
- board text added: "U$1"
- board text added: "U$2"
- board text added: "U$6"
- board text added: "VCNL4000"
- board text added: "jNode v3.2"
- board text removed: "+"
- board text removed: "-"
- board text removed: "jNode v3.1"

Commit message: add v33 jnode and cc3000 adapter board
Parts:
- removed IC6: MPL115A, mpl115:LGA8
- added U$3: MPL3115A2, jnode_v33:LGA8
- C5, C6: value 1µF -> 0.1µF
Connections:
- net GND: now also U$3.3; no longer IC6.3
- net N$10: now also U$3.2; no longer IC6.2
- net SCLK: now also U$3.7; no longer IC6.8
- net SDAT: now also U$3.8; no longer IC6.7
- net VSENS: now also U$3.1, U$3.4; no longer IC6.1, IC6.4, IC6.5
Routing:
- net VSENS: track 56.0 -> 45.4 mm
- net N$10: track 4.61 -> 0.00 mm
- net GND: track 39.9 -> 35.5 mm
- net SCLK: track 49.8 -> 47.7 mm
- net SDAT: track 45.2 -> 43.7 mm
