File: hardware/jnode/jnode_v33.sch (EAGLE design)
At the start: 59 parts, among them IC1 JENNIC_JN51XXSMDTH, IC2 ATMEGA32U4-AUQFN44, IC3 LTC3553, SW1 SONDER_H_VIBRATIONSSCHALTER, T1 DMP2104LP-7, U1 SHT21, X1 USBMICROB-XT

Commit message: add v33 jnode and cc3000 adapter board
Parts:
- removed R13: 2.2M, sparkfun:RESISTOR0402-RES
- removed R14: 1M, sparkfun:RESISTOR0402-RES
- removed SW1: SONDER_H_VIBRATIONSSCHALTER, jnode:SONDER_H_VIBRATIONSSCHALTER
- removed U$3: MPL3115A2, jnode_v33:MPL3115A2
- added C13: 0.1µF, sparkfun:CAP0402-CAP
- added C15: 10µF, sparkfun:CAP0603-CAP
- added IC6: MPL3115A2, jnode_v33:MPL3115A2
- added JP2: (no value), SparkFun-Passives:JUMPER-2SMD-NC
- added U4: LTC2942-1, PowerBoard.rpt:LTC2942-1
- BTN_PWR: DIGIKEY (none) -> P10852SCT-ND
- C1: DIGIKEY http://www.digikey.com/product-detail/en/JMK105BJ474KV-F/58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 -> 587-1230-1-ND
- C10: DIGIKEY http://search.digikey.com/scripts/DkSearch/dksus.dll?Detail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 -> 311-1014-1-ND; FARNELL http://de.farnell.com/multicomp/mcca000091/mlcc-0402-np0-50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 -> (none); TECO yes -> (none)
- C11: DIGIKEY http://www.digikey.com/product-detail/en/C0402C224K9PACTU/3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 -> 399-4886-1-ND
- C12, C14, C18, C4, C8: DIGIKEY http://search.digikey.com/scripts/DkSearch/dksus.dll?Detail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 -> 490-1318-1-ND; FARNELL http://de.farnell.com/multicomp/mcca000051/mlcc-04025v-16v-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 -> (none); TECO yes -> (none)
- C17, C22: DIGIKEY http://www.digikey.com/product-detail/en/C1608X6S0G106K080A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 -> 445-7454-1-ND
- C19, C20: value 10µF / near -> 10µF; DIGIKEY http://search.digikey.com/scripts/DkSearch/dksus.dll?Detail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 -> 445-7454-1-ND; FARNELL http://de.farnell.com/multicomp/mcca000517/mlcc-0603-x5r-6-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 -> (none); TECO yes -> (none)
- C2: value 100nF -> 0.1µF; DIGIKEY http://www.digikey.com/product-detail/en/C1005X5R0J104K050B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 -> 490-1318-1-ND
- C21: value 2.2µF / near -> 2.2µF; DIGIKEY http://search.digikey.com/scripts/DkSearch/dksus.dll?Detail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 -> 445-7396-1-ND; FARNELL http://de.farnell.com/multicomp/mcca000501/mlcc-0402-x5r-6-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 -> (none); TECO yes -> (none)
- C3: DIGIKEY http://www.digikey.com/product-detail/en/CL05A475MQ5NRNC/12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 -> 1276-1056-1-ND
- C5, C6: DIGIKEY (none) -> 490-1318-1-ND
- C7: DIGIKEY http://search.digikey.com/scripts/DkSearch/dksus.dll?Detail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 -> 490-1320-1-ND; FARNELL http://de.farnell.com/multicomp/mcca000500/mlcc-0402-x5r-6-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 -> (none); TECO yes -> (none)
- C9: DIGIKEY http://search.digikey.com/scripts/DkSearch/dksus.dll?Detail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 -> 445-7454-1-ND
- IC1: DIGIKEY http://search.digikey.com/de/de/products/JN5148%2F001M00T,5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 -> 616-1045-1-ND; FUTUREELECTRIC http://de.futureelectronics.com/de/technologies/semiconduct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 -> (none); PLACE NO -> no; TECO yes -> (none)
- IC2: DIGIKEY http://search.digikey.com/scripts/DkSearch/dksus.dll?Detail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 -> ATMEGA32U4-MU-ND
- IC3: DIGIKEY http://search.digikey.com/scripts/DkSearch/dksus.dll?Detail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 -> LTC3553EUD#PBF-ND
- JP1: PLACE (none) -> no
- L1: DIGIKEY (none) -> 445-6366-1-ND; FARNELL http://de.farnell.com/tdk/mlp2012s4r7mt/vielschicht-indukti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 -> (none)
- LED1: DIGIKEY http://search.digikey.com/scripts/DkSearch/dksus.dll?Detail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 -> 754-1128-1-ND; TECO yes -> (none)
- LED2: DIGIKEY http://search.digikey.com/scripts/DkSearch/dksus.dll?Detail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 -> 754-1127-1-ND; TECO yes -> (none)
- MICRO_SD1: value SENSOR_BOARD_MOLEX_47309-2651'NEW' -> MOLEX_47309-2651NEW; device teco_div:SENSOR_BOARD_MOLEX_47309-2651'NEW' -> jnode_v33:MOLEX_47309-2651NEW; DIGIKEY http://search.digikey.com/scripts/DkSearch/dksus.dll?Detail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 -> WM3974CT-ND; TECO yes -> (none)
- R10, R11: DIGIKEY http://search.digikey.com/scripts/DkSearch/dksus.dll?Detail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 -> RHM10.0KCDCT-ND
- R12: DIGIKEY http://www.digikey.com/product-detail/en/MCR01MRTF6800/RHM6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 -> RHM680CDCT-ND
- R18, R19: DIGIKEY http://search.digikey.com/scripts/DkSearch/dksus.dll?Detail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 -> 1276-3460-1-ND; FARNELL http://de.farnell.com/bourns/cr0603-jw-103elf/widerstand-06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 -> (none)
- R2: DIGIKEY http://search.digikey.com/scripts/DkSearch/dksus.dll?Detail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 -> 311-1.8KJRCT-ND; FARNELL http://de.farnell.com/vishay-draloric/crcw04021k80fkeahp/wi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 -> (none); TECO yes -> (none)
- R3: DIGIKEY http://www.digikey.com/product-search/en?FV=fff40001%2Cfff8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 -> RHM680CDCT-ND
- R4, R5: DIGIKEY http://search.digikey.com/scripts/DkSearch/dksus.dll?Detail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 -> 311-22JRCT-ND; FARNELL http://de.farnell.com/multicomp/mc-0-0625w-0402-1-22r/wider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 -> (none)
- R6: DIGIKEY http://search.digikey.com/scripts/DkSearch/dksus.dll?Detail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 -> RHM10.0KCDCT-ND; FARNELL http://de.farnell.com/bourns/cr0603-jw-103elf/widerstand-06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 -> (none); TECO yes -> (none)
- R7: DIGIKEY http://www.digikey.com/product-detail/en/RC0402JR-071M5L/31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 -> 311-1.5MJRCT-ND
- R8: DIGIKEY http://www.digikey.com/product-detail/en/RC0402FR-07560KL/3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 -> P560KLCT-ND
- R9: DIGIKEY http://www.digikey.com/product-detail/en/RC0402FR-071ML/311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 -> 311-1.00MLRCT-ND
- T1: DIGIKEY (none) -> DMP2104LPDICT-ND
- U1: device zittel:SHT21 -> jnode_v33:SHT21
- U2: ARROW (none) -> http://components.arrow.com/part/search/lsm9ds0; DIGIKEY http://www.digikey.de/product-detail/de/LSM9DS0TR/497-13902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 -> http://www.digikey.com/product-detail/en/LSM9DS0TR/497-1390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; MOUSER (none) -> http://de.mouser.com/ProductDetail/STMicroelectronics/LSM9D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
- U3: DIGIKEY http://www.digikey.com/product-detail/en/SFV5R-2STE1HLF/609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 -> 609-4330-1-ND
- U6: DIGIKEY (none) -> 478-5420-1-ND
- VCNL4010: DIGIKEY http://www.digikey.com/product-detail/en/VCNL4010-GS08/VCNL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 -> VCNL4010-GS08CT-ND
- X1: DIGIKEY http://search.digikey.com/scripts/DkSearch/dksus.dll?Detail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 -> H11635CT-ND
- renumbered U$1 to U3, U$2 to U2, U$6 to U6, VCNL4000 to VCNL4010
Connections:
- new net N$18: IC1.DIO12/TIM1_CAP, JP2.1
- new net SENSE+: C13.1, IC3.BAT, U4.SENSE+
- new net SENSE-: JP2.2, U3.1, U3.2, U4.SENSE-
- net BALLSW: no longer R13.1, SW1.2
- net GND: now also C13.2, C15.2, C2.2, IC6.GND, U4.GND; no longer C2.1, SW1.1, U$3.GND
- net N$10: now also IC6.CAP; no longer U$3.CAP
- net SCLK: now also IC6.SCL, U4.SCL; no longer U$3.SCL
- net SDAT: now also IC6.SDA, U4.SDA; no longer U$3.SDA
- net VCC: no longer C2.2, R14.1, U1.VDD
- net VOUT: no longer U3.1, U3.2
- net VSENS: now also C15.1, C2.1, IC6.VDD, IC6.VDDIO, U1.VDD; no longer R13.2, U$3.VDD, U$3.VDDIO
- net VSENS_OFF: no longer R14.2
Other:
- note added: "changes from 3.2: - connect BAT line - add Q-counter (plus res,cap) - reconnect hydro to VSENS - remove micro-vib - C1 replaced - remove superfluos R14 - change SFV5R order nr"
- note added: "digikey cart: http://www.digikey.de/short/5h5mj misses U1"
- note removed: "TODO: - re-connect BAT line!!!!"
- moved on the sheet: C2, C5
