File: hardware/jnode/jnode_v34.sch (EAGLE design)
At the start: 60 parts, among them IC1 JENNIC_JN51XXSMDTH, IC2 ATMEGA32U4-AUQFN44, IC3 LTC3553, IC6 MPL3115A2, T1 DMP2104LP-7, U1 SHT21, U2 LSM9D, U3 SFV5R, U4 LTC2942-1, U6 RESONATORPRQC-S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

Commit message: update jnode
Other:
- note added: "changes from v3.3: - fix GREEN LED connection - fix stepper"
- note removed: "changes from 3.2: - connect BAT line - add Q-counter (plus res,cap) - reconnect hydro to VSENS - remove micro-vib - C1 replaced - remove superfluos R14 - change SFV5R order nr"
- note removed: "changes to v3.3: - fix GREEN LED connection - fix stepper?"
Changed lines of the file:
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@@
 <text x="337.82" y="190.5" size="1.778" layer="98">VCNL_Address: 0010011x</text>
 <text x="340.36" y="238.76" size="1.778" layer="98">MPL_Address: 1100000x</text>
-<text x="134.62" y="152.4" size="1.778" layer="91">changes from 3.2:
- - connect BAT line
- - add Q-counter (plus res,cap)
- - reconnect  hydro to VSENS
- - remove micro-vib
- - C1 replaced
- - remove superfluos R14
- - change SFV5R order nr</text>
 <text x="243.84" y="233.68" size="1.778" layer="91">digikey cart:
 http://www.digikey.de/short/5h5mj
 misses U1</text>
-<text x="187.96" y="165.1" size="1.778" layer="91">changes to v3.3:
+<text x="187.96" y="165.1" size="1.778" layer="91">changes from v3.3:
  - fix GREEN LED connection
- - fix stepper?</text>
+ - fix stepper</text>
 </plain>
 <instances>
