File: hardware/jncc3000/jncc3000.brd (EAGLE design)
At the start: 17.6 x 29.1 mm, 8 parts

Commit message: add v33 jnode and cc3000 adapter board
Connections:
- new net VBAT: U$2.P$27, U1.VBAT_IN
- net +3V3: no longer U1.VBAT_IN
- net WL_RS232_RX: no longer U1.WL_RS232_RX
- net WL_RS232_TX: no longer U1.WL_RS232_TX
Routing:
- net WL_RS232_TX: track 15.3 -> 0.00 mm, vias 1 -> 0
- net WL_RS232_RX: track 12.1 -> 0.00 mm, vias 1 -> 0
- net VBAT: track 0.00 -> 8.16 mm
- net GND: track 16.1 -> 10.9 mm, vias 17 -> 33
- net WIFI_EN: track 15.9 -> 13.8 mm
- net +3V3: track 25.9 -> 27.9 mm, vias 0 -> 2
