File: hardware/jncc3000/jncc3000.sch (EAGLE design)
At the start: 8 parts, among them U4 NL17SZ125SOT553, X2 IPEX-20279-001E

Commit message: add v33 jnode and cc3000 adapter board
Parts:
- ANT1: MOUSER (none) -> http://de.mouser.com/ProductDetail/Johanson/2500AT44M0400E/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
- C3: MOUSER (none) -> http://de.mouser.com/ProductDetail/Vishay-Vitramon/VJ0603Y1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
- C4: MOUSER (none) -> http://de.mouser.com/ProductDetail/Johanson/251R14S0R8BV4T/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
- L1: MOUSER (none) -> http://de.mouser.com/ProductDetail/Johanson/L-14C3N3SV4T/?q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
- U1: MOUSER (none) -> http://de.mouser.com/ProductDetail/Texas-Instruments/CC3000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
- U4: MOUSER (none) -> http://de.mouser.com/ProductDetail/ON-Semiconductor/NL17SZ1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
Connections:
- new net VBAT: U$2.DIO12/TIM1_CAP, U1.VBAT_IN
- net +3V3: no longer U1.VBAT_IN
- net WL_RS232_RX: no longer U1.WL_RS232_RX
- net WL_RS232_TX: no longer U1.WL_RS232_TX
Changed lines of the file:
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@@
 <part name="U1" library="jncc3000.lbrjncc3000" deviceset="CC3000" device="">
 <attribute name="DIGIKEY" value="www.digikey.de/product-detail/en/CC3000MODR/296-35512-1-ND/3768439"/>
+<attribute name="MOUSER" value="http://de.mouser.com/ProductDetail/Texas-Instruments/CC3000MOD/?qs=sGAEpiMZZMul4LbMdexInYO9dzLxESeK"/>
 </part>
 <part name="GND5" library="SparkFun" deviceset="GND" device=""/>
@@
 <part name="C3" library="rcl" deviceset="C-EU" device="C0603" value="100nF">
 <attribute name="DIGIKEY" value="www.digikey.de/product-detail/en/CC0603KRX7R8BB104/311-1341-1-ND/2103125"/>
+<attribute name="MOUSER" value="http://de.mouser.com/ProductDetail/Vishay-Vitramon/VJ0603Y104JXJCW1BC/?qs=sGAEpiMZZMs0AnBnWHyRQAR7at33PD0%252bJG6E%252bZ2ATD0%3d"/>
 </part>
 <part name="P+1" library="SparkFun" deviceset="3.3V" device="" value="+3V3"/>
@@
 <part name="ANT1" library="Spark" deviceset="AT8010" device="">
 <attribute name="DIGIKEY" value="www.digikey.de/product-detail/en/2500AT44M0400E/712-1403-1-ND/1840081"/>
+<attribute name="MOUSER" value="http://de.mouser.com/ProductDetail/Johanson/2500AT44M0400E/?qs=%2fha2pyFadugpD5gBUDGQSiDxg6DUc4t7HJxRbOdSf%2fyD3Zvh3vVhxQ%3d%3d"/>
 </part>
 <part name="GND21" library="SparkFun" deviceset="GND" device=""/>
 <part name="U4" library="jncc3000.lbrjncc3000" deviceset="NL17SZ125" device="SOT553" value="">
 <attribute name="DIGIKEY" value="www.digikey.de/product-detail/en/NL17SZ125XV5T2G/NL17SZ125XV5T2GOSCT-ND/3462428"/>
+<attribute name="MOUSER" value="http://de.mouser.com/ProductDetail/ON-Semiconductor/NL17SZ125XV5T2G/?qs=%2fha2pyFadugaeFY%2fWCqy5e2mGAS%252bZ6GlBMnp3M0qQT2RP75tHTbjNQ%3d%3d"/>
 </part>
 <part name="GND2" library="SparkFun" deviceset="GND" device=""/>
@@
 <attribute name="COMMENT" value="RF Inductor"/>
 <attribute name="DIGIKEY" value="www.digikey.de/product-detail/en/L-14C3N3SV4T/712-1428-1-ND/1914878"/>
+<attribute name="MOUSER" value="http://de.mouser.com/ProductDetail/Johanson/L-14C3N3SV4T/?qs=%2fha2pyFaduhrzBAYMc2Wa%252b3wfGy6CaphxWSEKt2XW6iFpd4j0hTO4g%3d%3d"/>
 </part>
 <part name="C4" library="rcl" deviceset="C-EU" device="C0603" value="0.8pF">
 <attribute name="COMMENT" value="RF Capacitor"/>
 <attribute name="DIGIKEY" value="www.digikey.de/product-detail/en/251R14S0R8BV4T/712-1305-1-ND/1786767"/>
+<attribute name="MOUSER" value="http://de.mouser.com/ProductDetail/Johanson/251R14S0R8BV4T/?qs=%2fha2pyFaduiSPVteKT%2fHqbo88L%252bTOfWWrsdG4xq6eKjM4bWhxYlobA%3d%3d"/>
 </part>
 <part name="U$2" library="jncc3000.lbrjncc3000" deviceset="JENNIC_JN51XX" device="TH" value="">
@@
 <instance part="U1" gate="G$1" x="180.34" y="119.38">
 <attribute name="DIGIKEY" x="180.34" y="119.38" size="1.778" layer="96" display="off"/>
+<attribute name="MOUSER" x="180.34" y="119.38" size="1.778" layer="96" display="off"/>
 </instance>
 <instance part="GND5" gate="1" x="203.2" y="152.4"/>
@@
 <attribute name="VALUE" x="146.304" y="58.801" size="1.778" layer="96"/>
 <attribute name="DIGIKEY" x="144.78" y="63.5" size="1.778" layer="96" display="off"/>
+<attribute name="MOUSER" x="144.78" y="63.5" size="1.778" layer="96" display="off"/>
 </instance>
 <instance part="P+1" gate="G$1" x="233.68" y="78.74" rot="R180"/>
@@
 <instance part="ANT1" gate="G$1" x="133.35" y="172.72" rot="R90">
 <attribute name="DIGIKEY" x="133.35" y="172.72" size="1.778" layer="96" rot="R90" display="off"/>
+<attribute name="MOUSER" x="133.35" y="172.72" size="1.778" layer="96" rot="R90" display="off"/>
 </instance>
 <instance part="GND21" gate="1" x="152.4" y="153.67"/>
 <instance part="U4" gate="G$1" x="203.2" y="53.34">
 <attribute name="DIGIKEY" x="203.2" y="53.34" size="1.778" layer="96" display="off"/>
+<attribute name="MOUSER" x="203.2" y="53.34" size="1.778" layer="96" display="off"/>
 </instance>
 <instance part="GND2" gate="1" x="198.12" y="43.18"/>
@@
 <attribute name="DIGIKEY" x="165.1" y="172.72" size="1.778" layer="96" rot="R90" display="off"/>
 <attribute name="COMMENT" x="165.1" y="172.72" size="1.778" layer="96" rot="R90" display="off"/>
+<attribute name="MOUSER" x="165.1" y="172.72" size="1.778" layer="96" rot="R90" display="off"/>
 </instance>
 <instance part="C4" gate="G$1" x="152.4" y="165.1" smashed="yes">
@@
 <attribute name="DIGIKEY" x="152.4" y="165.1" size="1.778" layer="96" display="off"/>
 <attribute name="COMMENT" x="152.4" y="165.1" size="1.778" layer="96" display="off"/>
+<attribute name="MOUSER" x="152.4" y="165.1" size="1.778" layer="96" display="off"/>
 </instance>
 <instance part="U$2" gate="G$1" x="40.64" y="137.16">
@@
 <pinref part="U1" gate="G$1" pin="VIO_HOST"/>
 <wire x1="213.36" y1="116.84" x2="233.68" y2="116.84" width="0.1524" layer="91"/>
-<pinref part="U1" gate="G$1" pin="VBAT_IN"/>
-<wire x1="213.36" y1="106.68" x2="233.68" y2="106.68" width="0.1524" layer="91"/>
-<wire x1="233.68" y1="116.84" x2="233.68" y2="106.68" width="0.1524" layer="91"/>
 <pinref part="P+1" gate="G$1" pin="3.3V"/>
-<wire x1="233.68" y1="106.68" x2="233.68" y2="78.74" width="0.1524" layer="91"/>
-<junction x="233.68" y="106.68"/>
+<wire x1="233.68" y1="116.84" x2="233.68" y2="78.74" width="0.1524" layer="91"/>
 </segment>
 <segment>
@@
 <net name="WL_RS232_TX" class="0">
 <segment>
-<pinref part="U1" gate="G$1" pin="WL_RS232_TX"/>
-<wire x1="144.78" y1="116.84" x2="139.7" y2="116.84" width="0.1524" layer="91"/>
-</segment>
-<segment>
 <pinref part="U$2" gate="G$1" pin="DIO7/RXD0"/>
 <wire x1="27.94" y1="99.06" x2="17.78" y2="99.06" width="0.1524" layer="91"/>
@@
 <net name="WL_RS232_RX" class="0">
 <segment>
-<pinref part="U1" gate="G$1" pin="WL_RS232_RX"/>
-<wire x1="144.78" y1="111.76" x2="137.16" y2="111.76" width="0.1524" layer="91"/>
-</segment>
-<segment>
 <pinref part="U$2" gate="G$1" pin="DIO6/TXD0"/>
 <wire x1="27.94" y1="101.6" x2="17.78" y2="101.6" width="0.1524" layer="91"/>
@@
 </segment>
 </net>
+<net name="VBAT" class="0">
+<segment>
+<pinref part="U1" gate="G$1" pin="VBAT_IN"/>
+<wire x1="213.36" y1="106.68" x2="223.52" y2="106.68" width="0.1524" layer="91"/>
+</segment>
+<segment>
+<pinref part="U$2" gate="G$1" pin="DIO12/TIM1_CAP"/>
+<wire x1="86.36" y1="93.98" x2="99.06" y2="93.98" width="0.1524" layer="91"/>
+</segment>
+</net>
